Commit message: 0120.1已完成初步控制挖掘机（除swing）

File: src/excavator_sim/urdf/excavator.urdf.xacro (robot description, xacro)
@@ -2,10 +2,10 @@
 <robot name="excavator" xmlns:xacro="http://www.ros.org/wiki/xacro">
   <!-- 参数定义 -->
-  <xacro:property name="chassis_length" value="2.0"/>
+  <xacro:property name="chassis_length" value="2.5"/>
   <xacro:property name="chassis_width" value="1.2"/>
   <xacro:property name="chassis_height" value="0.4"/>
   <xacro:property name="track_width" value="0.3"/>
   <xacro:property name="track_radius" value="0.25"/>
-  <xacro:property name="cabin_length" value="1.0"/>
+  <xacro:property name="cabin_length" value="1.6"/>
   <xacro:property name="cabin_width" value="0.8"/>
   <xacro:property name="cabin_height" value="1.0"/>
@@ -85,10 +85,8 @@
     </inertial>
   </link>
-  <joint name="left_track_joint" type="continuous">
+  <joint name="left_track_joint" type="fixed">
     <parent link="chassis"/>
     <child link="left_track"/>
     <origin xyz="0 ${chassis_width/2 + track_width/2} ${-chassis_height/2}" rpy="0 0 0"/>
-    <axis xyz="0 1 0"/>
-    <dynamics damping="10.0" friction="5.0"/>
   </joint>
   <!-- 右履带 -->
@@ -110,10 +108,8 @@
     </inertial>
   </link>
-  <joint name="right_track_joint" type="continuous">
+  <joint name="right_track_joint" type="fixed">
     <parent link="chassis"/>
     <child link="right_track"/>
     <origin xyz="0 ${-chassis_width/2 - track_width/2} ${-chassis_height/2}" rpy="0 0 0"/>
-    <axis xyz="0 1 0"/>
-    <dynamics damping="10.0" friction="5.0"/>
   </joint>
   <!-- ========== 座舱回转平台 ========== -->
@@ -143,5 +139,5 @@
     <origin xyz="0 0 ${chassis_height/2}" rpy="0 0 0"/>
     <axis xyz="0 0 1"/>
-    <dynamics damping="100.0" friction="10.0"/>
+    <dynamics damping="10.0" friction="10.0"/>
     <limit effort="10000" velocity="1.0"/>
   </joint>
@@ -172,6 +168,6 @@
     <origin xyz="${cabin_length/2} 0 ${cabin_height}" rpy="0 0 0"/>
     <axis xyz="0 1 0"/>
-    <dynamics damping="50.0" friction="5.0"/>
-    <limit lower="-0.5" upper="1.2" effort="50000" velocity="0.5"/>
+    <dynamics damping="100.0" friction="10.0"/>
+    <limit lower="-1.5" upper="0.5" effort="1000000" velocity="0.5"/>
   </joint>
   <!-- ========== 小臂 (Arm/Stick) ========== -->
@@ -201,6 +197,6 @@
     <origin xyz="${boom_length} 0 0" rpy="0 0 0"/>
     <axis xyz="0 1 0"/>
-    <dynamics damping="30.0" friction="3.0"/>
-    <limit lower="-2.5" upper="0.5" effort="30000" velocity="0.6"/>
+    <dynamics damping="100.0" friction="100.0"/>
+    <limit lower="-1.0" upper="2.5" effort="30000" velocity="0.6"/>
   </joint>
   <!-- ========== 铲斗 (Bucket) ========== -->
@@ -230,5 +226,5 @@
     <origin xyz="${arm_length} 0 0" rpy="0 0 0"/>
     <axis xyz="0 1 0"/>
-    <dynamics damping="20.0" friction="2.0"/>
+    <dynamics damping="50.0" friction="50.0"/>
     <limit lower="-1.5" upper="1.5" effort="15000" velocity="0.8"/>
   </joint>

Commit message: 0121.1已实现键盘控制；能控制写字但效果不好

File: src/excavator_sim/urdf/excavator.urdf.xacro (robot description, xacro)
@@ -139,6 +139,6 @@
     <origin xyz="0 0 ${chassis_height/2}" rpy="0 0 0"/>
     <axis xyz="0 0 1"/>
-    <dynamics damping="10.0" friction="10.0"/>
-    <limit effort="10000" velocity="1.0"/>
+    <dynamics damping="5.0" friction="1.0"/>
+    <!-- <limit effort="10000" velocity="1.0"/> -->
   </joint>
   <!-- ========== 大臂 (Boom) ========== -->
@@ -250,21 +250,13 @@
   </joint>
   <!-- ========== Gazebo 插件 ========== -->
-  <!-- 差速驱动控制器 -->
+  <!-- 平面移动插件 -->
   <gazebo>
-    <plugin name="differential_drive_controller" filename="libgazebo_ros_diff_drive.so">
-      <legacyMode>false</legacyMode>
-      <alwaysOn>true</alwaysOn>
-      <updateRate>50</updateRate>
-      <leftJoint>left_track_joint</leftJoint>
-      <rightJoint>right_track_joint</rightJoint>
-      <wheelSeparation>${chassis_width + track_width}</wheelSeparation>
-      <wheelDiameter>${track_radius * 2}</wheelDiameter>
-      <torque>1000</torque>
-      <commandTopic>cmd_vel</commandTopic>
+    <plugin name="planar_move_controller" filename="libgazebo_ros_planar_move.so">
+      <commandTopic>/excavator/cmd_vel</commandTopic>
       <odometryTopic>odom</odometryTopic>
       <odometryFrame>odom</odometryFrame>
       <robotBaseFrame>base_footprint</robotBaseFrame>
-      <publishWheelTF>true</publishWheelTF>
-      <publishWheelJointState>true</publishWheelJointState>
+      <odometryRate>50.0</odometryRate>
+      <publishOdometryTf>true</publishOdometryTf>
     </plugin>
   </gazebo>

Commit message: 0122.1未有改善，存档

File: src/excavator_sim/urdf/excavator.urdf.xacro (robot description, xacro)
@@ -58,6 +58,6 @@
     </collision>
     <inertial>
-      <mass value="5000"/>
-      <xacro:box_inertia m="5000" x="${chassis_length}" y="${chassis_width}" z="${chassis_height}"/>
+      <mass value="8000"/>
+      <xacro:box_inertia m="8000" x="${chassis_length}" y="${chassis_width}" z="${chassis_height}"/>
     </inertial>
   </link>

Commit message: 0225.1使用了pykdl

File: src/excavator_sim/urdf/excavator.urdf.xacro (robot description, xacro)
@@ -169,5 +169,5 @@
     <axis xyz="0 1 0"/>
     <dynamics damping="100.0" friction="10.0"/>
-    <limit lower="-1.5" upper="0.5" effort="1000000" velocity="0.5"/>
+    <limit lower="-2.0" upper="1.5" effort="1000000" velocity="0.5"/>
   </joint>
   <!-- ========== 小臂 (Arm/Stick) ========== -->
@@ -198,5 +198,5 @@
     <axis xyz="0 1 0"/>
     <dynamics damping="100.0" friction="100.0"/>
-    <limit lower="-1.0" upper="2.5" effort="30000" velocity="0.6"/>
+    <limit lower="-2.8" upper="2.5" effort="30000" velocity="0.6"/>
   </joint>
   <!-- ========== 铲斗 (Bucket) ========== -->
@@ -227,5 +227,5 @@
     <axis xyz="0 1 0"/>
     <dynamics damping="50.0" friction="50.0"/>
-    <limit lower="-1.5" upper="1.5" effort="15000" velocity="0.8"/>
+    <limit lower="-3.14" upper="3.14" effort="15000" velocity="0.8"/>
   </joint>
   <!-- 铲斗末端（用于轨迹跟踪） -->
